File: Kicad/L235-Analog-Processor.kicad_sch (KiCad schematic)
At the start: 346 parts, among them J1 Input A, J10 Half Wave A + -B, J12 CV Select, J13 CV Select, J14 Conn_01x20_Pin, J16 Full-Wave Rectifier A, J17 Half-Wave Rectifier A, J18 √(A²+B²), J19 Conn_01x20_Socket, J2 Input B, J20 Conn_01x05_Socket, J21 Conn_01x05_Pin, J22 Conn_01x05_Socket, J23 Conn_01x05_Pin, J3 Function IN, J4 ( 10A / |B| ) / ( A * B / 10 ), J5 Output F(x), J6 Power, J7 Full-Wave Rectifier B, J8 A - B, J9 Negative Half-Wave Rectifier B, U1 TL082, U10 TL082, U11 TL082, U12 TL082, U13 TL084, U14 RC4580, U15 TL082, U16 AD633ARZ-RL, U17 TL082, U19 74HC148, U2 TL082, U20 LM339, U21 LM339, U22 CD4051, U23 CD4051, U24 CD4051, U25 CD4051, U26 CD4051, U27 CD4051, U28 CD4051, U29 LM339, U3 TL082, U30 LM339, U31 74HC148, U32 DG4051E, U33 DG4051E, U34 DG4051E, U35 DG4051E, U36 LM78M05_TO252, U37 TL082, U39 CD4051, U4 TL082, U40 CD4051, U5 TL082, U6 TL082, U7 TL082, U8 TL082, U9 TL082

Commit message: Replaced 4051 with DG408 to allow negative -10V voltages
Parts:
- U22, U23, U24, U25, U26, U27, U28: value CD4051 -> DG408
- U32, U33, U34, U35: value DG4051E -> DG408
Changed lines of the file:
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@@
       (effects (font (size 1.27 1.27)))
     )
-    (property "Value" "CD4051" (at 181.61 515.7821 0)
+    (property "Value" "DG408" (at 181.61 515.7821 0)
       (effects (font (size 1.27 1.27)))
     )
@@
       (effects (font (size 1.27 1.27)))
     )
-    (property "Value" "DG4051E" (at 426.72 567.8521 0)
+    (property "Value" "DG408" (at 426.72 567.8521 0)
       (effects (font (size 1.27 1.27)))
     )
@@
       (effects (font (size 1.27 1.27)))
     )
-    (property "Value" "CD4051" (at 181.61 647.8621 0)
+    (property "Value" "DG408" (at 181.61 647.8621 0)
       (effects (font (size 1.27 1.27)))
     )
@@
       (effects (font (size 1.27 1.27)))
     )
-    (property "Value" "CD4051" (at 181.61 712.6321 0)
+    (property "Value" "DG408" (at 181.61 712.6321 0)
       (effects (font (size 1.27 1.27)))
     )
@@
       (effects (font (size 1.27 1.27)))
     )
-    (property "Value" "DG4051E" (at 426.72 631.9871 0)
+    (property "Value" "DG408" (at 426.72 631.9871 0)
       (effects (font (size 1.27 1.27)))
     )
@@
       (effects (font (size 1.27 1.27)))
     )
-    (property "Value" "CD4051" (at 181.61 583.0921 0)
+    (property "Value" "DG408" (at 181.61 583.0921 0)
       (effects (font (size 1.27 1.27)))
     )
@@
       (effects (font (size 1.27 1.27)))
     )
-    (property "Value" "DG4051E" (at 426.72 503.0821 0)
+    (property "Value" "DG408" (at 426.72 503.0821 0)
       (effects (font (size 1.27 1.27)))
     )
@@
       (effects (font (size 1.27 1.27)))
     )
-    (property "Value" "CD4051" (at 181.61 845.9821 0)
+    (property "Value" "DG408" (at 181.61 845.9821 0)
       (effects (font (size 1.27 1.27)))
     )
@@
       (effects (font (size 1.27 1.27)))
     )
-    (property "Value" "DG4051E" (at 426.72 698.0271 0)
+    (property "Value" "DG408" (at 426.72 698.0271 0)
       (effects (font (size 1.27 1.27)))
     )
@@
       (effects (font (size 1.27 1.27)))
     )
-    (property "Value" "CD4051" (at 181.61 447.2021 0)
+    (property "Value" "DG408" (at 181.61 447.2021 0)
       (effects (font (size 1.27 1.27)))
     )
@@
       (effects (font (size 1.27 1.27)))
     )
-    (property "Value" "CD4051" (at 181.61 781.2121 0)
+    (property "Value" "DG408" (at 181.61 781.2121 0)
       (effects (font (size 1.27 1.27)))
     )
