File: Kicad/L235-Analog-Processor.kicad_sch (KiCad schematic)
At the start: 346 parts, among them J1 Input A, J10 Half Wave A + -B, J12 CV Select, J13 CV Select, J14 Conn_01x20_Pin, J16 Full-Wave Rectifier A, J17 Half-Wave Rectifier A, J18 √(A²+B²), J19 Conn_01x20_Socket, J2 Input B, J20 Conn_01x05_Socket, J21 Conn_01x05_Pin, J22 Conn_01x05_Socket, J23 Conn_01x05_Pin, J3 Function IN, J4 ( 10A / |B| ) / ( A * B / 10 ), J5 Output F(x), J6 Power, J7 Full-Wave Rectifier B, J8 A - B, J9 Negative Half-Wave Rectifier B, U1 TL082, U10 TL082, U11 TL082, U12 TL082, U13 TL084, U14 RC4580, U15 TL082, U16 AD633ARZ-RL, U17 TL082, U19 74HC148, U2 TL082, U20 LM339, U21 LM339, U22 DG408, U23 DG408, U24 DG408, U25 DG408, U26 DG408, U27 DG408, U28 DG408, U29 LM339, U3 TL082, U30 LM339, U31 74HC148, U32 DG408, U33 DG408, U34 DG408, U35 DG408, U36 LM78M05_TO252, U37 TL082, U39 CD4051, U4 TL082, U40 CD4051, U5 TL082, U6 TL082, U7 TL082, U8 TL082, U9 TL082

Commit message: Fixed attenuverter circuit after breadboard testing
Parts:
- removed RV1: 50k, Potentiometer_THT:Potentiometer_Bourns_3339H_Vertical, symbol Device:R_Potentiometer_Trim
- added C43, C79: 100nF, Capacitor_SMD:C_0402_1005Metric, symbol Device:C
- added D46, D47, D48, D49, D50, D51: U21,5, Diode_SMD:D_SOD-123, symbol Device:D
- added R136, R144, R146, R149, R150, R163: 220k, Resistor_SMD:R_0402_1005Metric, symbol Device:R
- added R139, R160, R162: 1k, Resistor_SMD:R_0402_1005Metric, symbol Device:R
- added R140, R141, R142, R143, R145, R165: 100k, Resistor_SMD:R_0402_1005Metric, symbol Device:R
- added R147, R148: 2k2, Resistor_SMD:R_0402_1005Metric, symbol Device:R
- added R151, R161: 100, Resistor_SMD:R_0402_1005Metric, symbol Device:R
- added R159: 3k, Resistor_SMD:R_0402_1005Metric, symbol Device:R
- added R164: 2k, Resistor_SMD:R_0402_1005Metric, symbol Device:R
- added R166: 4k7, Resistor_SMD:R_0402_1005Metric, symbol Device:R
- added R168, R169, R171, R172, R173: 10k, Resistor_SMD:R_0402_1005Metric, symbol Device:R
- added R170: 500, Resistor_SMD:R_0402_1005Metric, symbol Device:R
- added RV1: 100k, Potentiometer_THT:Potentiometer_Bourns_3339H_Vertical, symbol Device:R_Potentiometer
- added RV14, RV16: 100k, Potentiometer_THT:Potentiometer_Alpha_RD901F-40-00D_Single_Vertical, symbol Device:R_Potentiometer
- added SW1: SW_SPDT, symbol Switch:SW_SPDT
- added U18, U38: TL082, Package_SO:SO-8_3.9x4.9mm_P1.27mm, symbol Amplifier_Operational:TL082
- added U42: TL082, Package_SO:SOIC-8_3.9x4.9mm_P1.27mm, symbol Amplifier_Operational:TL082
- added U43: LM339, Package_SO:SOIC-14_3.9x8.7mm_P1.27mm, symbol Comparator:LM339
- R10: value 10k -> 500
- R135, R4: value 100k -> 47k
- R137, R2: value 220k -> 100k
- R18: value 300k -> 220k
Connections:
- net +12V: now also R10.1, R146.1, R150.1, R159.2, R164.1, R165.2, R170.1, RV1.1, RV14.1
- net -12V: now also R144.1, R149.1, R163.1, RV1.3, RV14.3
- net A: now also D47.2 (A), D49.1 (K), R140.1, R143.2, R168.1
- net B: now also D48.2 (A), D50.1 (K), R141.1, R142.2, R169.1
- net GND: now also R134.1, R82.1, C43.1, C79.1, R139.1, R148.1, R166.2, RV16.2, RV16.3, SW1.1 (A), U18.3 (+); no longer R10.1, U28.1 (X4), U28.12 (X3), U28.13 (X0), U28.14 (X1), U28.15 (X2), U28.5 (X5)
- net at R39.1, R82.2, U15.3 (+): now also RV10.2
- net at R137.1, RV15.2: now also C43.2
- net at R9.2, U4.3 (+): now also R11.2; no longer R10.2
- net at R12.1, U4.2 (-): now also R173.2; no longer R11.2
- net at R18.2: now also RV1.2
- net at R133.1, R134.2, U1.3 (+): now also RV9.2
- net at R2.1, RV13.2: now also C79.2
- new net: R165.1, RV16.1, U18.6 (-)
- new net: R147.1, U18.7
- new net: D51.1 (K), R151.1, U38.1
- new net: R169.2, R171.1, U42.2 (-)
- new net: R162.1, R164.2, U43.10 (-)
- new net: R160.1, R162.2, U43.6 (-)
- new net: D46.2 (A), R161.1, U38.7
- new net: R168.2, R172.2, U42.3 (+)
- new net: D49.2 (A), D50.2 (A), R150.2, U38.3 (+)
- new net: R142.1, R143.1, R144.2, U18.2 (-)
- new net: R145.1, U18.1
- new net: R159.1, R160.2, U43.4 (-)
- new net: D47.1 (K), D48.1 (K), R149.2, U38.5 (+)
- new net: R136.2, RV14.2
- new net A + B: R171.2, U42.1
- new net C: SW1.3 (C)
- new net Max: R151.2
- new net Min: R161.2
- new net Modulator: D46.1 (K), D51.2 (A), R140.2, R141.2, R145.2, R146.2, R163.2, R172.1, R173.1, SW1.2 (B), U18.5 (+), U38.2 (-), U38.6 (-)
- new net Squarer_IN: U43.11 (+), U43.5 (+), U43.7 (+)
- new net Squarer_OUT: R10.2, R166.1, R170.2, U43.1, U43.13, U43.2
- new net Volt_ref_Y: R136.1, R139.2, U28.1 (X4), U28.12 (X3), U28.13 (X0), U28.14 (X1), U28.15 (X2), U28.5 (X5)
- new net XOR: R147.2, R148.2
Other:
- note added: "-10/+10V"
- note added: "-50/+50mV (using 100k as original will make it 110mV)"
- note added: "3 Band Comparator (Min/Max/Zero)"
- note added: "470k on datasheet example"
- note added: "Analog XOR"
- note added: "BIAS -10/+10V"
- note added: "INPUT -5/+5V"
- note added: "Initial MAX limit (3-5V)"
- note added: "MIN limit -12 to +5V Threshold"
- note added: "Max"
- note added: "Min"
- note added: "Subtract"
- note added: "Sum"
- note removed: "470k on original"
- moved on the sheet: R11, R12, R9, RV10, RV9, U4A
